File: hardware/368255-2-connector/368255-2.sch (KiCad schematic (older format))
At the start: 41 parts, among them P1 CONN_3, P10 CONN_1, P11 CONN_1, P12 CONN_1, P13 CONN_3, P14 CONN_3, P15 CONN_1, P16 CONN_1, P17 CONN_1, P18 CONN_1, P19 CONN_1, P2 CONN_3, P20 CONN_1, P21 CONN_1, P22 CONN_1, P23 CONN_1, P24 CONN_1, P25 368255-2, P26 CONN_8, P27 CONN_8, P28 CONN_8, P29 CONN_8, P3 CONN_1, P30 CONN_8, P31 CONN_8, P32 CONN_8, P33 CONN_8, P34 CONN_8, P35 CONN_8, P36 CONN_8, P37 CONN_8, P38 CONN_1, P39 CONN_1, P4 CONN_1, P40 CONN_1, P41 CONN_1, P5 CONN_1, P6 CONN_1, P7 CONN_1, P8 CONN_1, P9 CONN_1

Commit message: manual sync
Parts:
- removed P1, P13, P14, P2: CONN_3, SIL-3, symbol CONN_3
- removed P26, P27, P28, P29, P30, P31, P36, P37: CONN_8, SIL-8, symbol CONN_8
- removed P3, P38, P39, P4, P40, P41, P5: CONN_1, SIL-1, symbol CONN_1
- added P13, P14, P25, P26, P27, P28, P29, P30, P31, P36, P37: CONN_1, symbol CONN_1
- added P2, P3, P4, P5: CONN_19, symbol CONN_19
- P10, P11, P12, P15, P16, P17, P18, P19, P20, P21, P22, P23, P24, P6, P7, P8, P9: footprint SIL-1 -> (none)
- P32, P33, P34, P35: footprint SIL-8 -> (none)
- renumbered P25 to P1
Connections:
- wire segments 65 -> 139
Other:
- moved on the sheet: P1A
