File: hardware/power_supply_kb1gtt/PWR_buck_12V_switcher.kicad_pcb (KiCad board)
At the start: 2 copper layers, 38.1 x 38.7 mm, 19 parts, among them P1 CONN_2, P2 CONN_1, P3 CONN_2, Q1 MOS_PRO, U1 LM2596

Commit message: auto-sync
Parts:
- added P4: CONN_1, SIL-1, F.Cu at (163.8, 109.2)
- added Q2: 200V, m-pad-2.1-TO-263AB, B.Cu at (174.6, 120.7)
- added R3: 100k, SM0805, B.Cu at (188.0, 120.7)
- C1: value 470uF 25V -> 330uF 35V
- D1: value ZENERSMALL -> 7.5V
- D2: value TVS -> 15V
- D3: value TVS -> 24V
- D5: value GREEN -> LED-grn
- F1: value 3.5A -> 5A
- Q1: value MOS_PRO -> 30V
- R1: value 1k -> 39k
- turned D2 to 90 degrees
Connections:
- D2 pad 2: /VBAT -> /Vs1
- Q1 pad 3: /Vf -> /Vs2
Routing:
- net /Vs1: track 0.00 -> 26.6 mm
- net /Vs2: track 0.00 -> 8.95 mm, vias 0 -> 1
- net /Vf: track 17.1 -> 11.1 mm
- net /VBAT: track 27.3 -> 24.4 mm
Other:
- board text added: "TEST POINT P2"
- board text added: "for rusEFI https://sourceforge.net/p/rusefi/"
- board text removed: "P2 TEST POINT"
- board text removed: "for rusEFI http://code.google.com/p/daecu/"

Commit message: auto-sync
Parts:
- added L3: 38uH, SM100uH, B.Cu at (168.3, 106.0)
- D2: value 15V -> 14V
- D3: moved to B.Cu
- Q1: value 30V -> 20V
- moved D3 23.4 mm to (167.4, 97.3), turned to 180 degrees
Connections:
- D1 pad 2: /VBAT -> Net-(D1-Pad2)
- P4 pad 1: /VBAT -> Net-(D1-Pad2)
- Q1 pad 2: /VBAT -> Net-(D1-Pad2)
Routing:
- net Net-(D1-Pad2): track 0.00 -> 12.7 mm
- net /VBAT: track 24.4 -> 22.6 mm, vias 0 -> 1
- net GND: track 83.0 -> 82.2 mm
Other:
- rule via_min_drill: 0.508 -> 0.3

Commit message: auto-sync
Parts:
- added P5: CONN_1, SIL-1, B.Cu at (163.6, 99.2)
- moved F1 0.76 mm to (177.8, 127.8)
- moved P1 0.25 mm to (168.0, 130.2)
Routing:
- net /VBAT: track 22.6 -> 27.2 mm
Other:
- net class 5A EXT 200V added: clearance 1.016, trace_width 1.38176, via_dia 1.651, via_drill 1.143
- board text added: "R0.4"
- board text removed: "R0.3"
Changed lines of the file:
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@@
 (kicad_pcb (version 4) (host pcbnew 4.0.1-stable)
   (general
-    (links 39)
+    (links 40)
     (no_connects 0)
-    (area 160.02 92.71 212.697787 141.986)
+    (area 159.457572 92.71 212.697787 141.986)
     (thickness 1.6002)
     (drawings 19)
-    (tracks 121)
+    (tracks 125)
     (zones 0)
-    (modules 23)
+    (modules 24)
     (nets 13)
   )
@@
     (35 F.Paste user)
     (36 B.SilkS user)
-    (37 F.SilkS user hide)
+    (37 F.SilkS user)
     (38 B.Mask user)
     (39 F.Mask user)
@@
     (pad_to_mask_clearance 0.254)
     (aux_axis_origin 0 0)
-    (visible_elements 7FFFFF3F)
+    (visible_elements 7FFFFF7F)
     (pcbplotparams
-      (layerselection 0x00030_80000001)
+      (layerselection 0x010fc_80000001)
       (usegerberextensions true)
       (excludeedgelayer true)
@@
     (add_net /OUT)
     (add_net /VBAT)
-    (add_net /Vf)
-    (add_net /Vin)
     (add_net /Vs1)
     (add_net /Vs2)
     (add_net GND)
     (add_net "Net-(D1-Pad2)")
+  )
+  (net_class "5A EXT 200V" ""
+    (clearance 1.016)
+    (trace_width 1.38176)
+    (via_dia 1.651)
+    (via_drill 1.143)
+    (uvia_dia 0.762)
+    (uvia_drill 0.254)
+    (add_net /Vf)
+    (add_net /Vin)
   )
   (net_class "5A INT" ""
@@
     (uvia_drill 0.254)
   )
+  (module SIL-1 (layer Back-ext)
+    (at 163.576 99.187)
+    (descr "Connecteurs 1 pin")
+    (tags "CONN DEV")
+    (fp_text reference P5 (at 0 2.54) (layer B.SilkS)
+      (effects (font (size 1.72974 1.08712) (thickness 0.27178)) (justify mirror))
+    )
+    (fp_text value CONN_1 (at 0 2.54) (layer B.SilkS) hide
+      (effects (font (size 1.524 1.016) (thickness 0.254)) (justify mirror))
+    )
+    (fp_line (start -1.27 -1.27) (end 1.27 -1.27) (layer B.SilkS) (width 0.3175))
+    (fp_line (start -1.27 1.27) (end 1.27 1.27) (layer B.SilkS) (width 0.3175))
+    (fp_line (start -1.27 -1.27) (end -1.27 1.27) (layer B.SilkS) (width 0.3048))
+    (fp_line (start 1.27 1.27) (end 1.27 -1.27) (layer B.SilkS) (width 0.3048))
+    (pad 1 thru_hole rect (at 0 0) (size 1.397 1.397) (drill 0.8128) (layers *.Cu *.Mask B.SilkS)
+      (net 4 /VBAT))
+  )
   (module SM100uH (layer Back-ext)
     (at 168.275 106.045 90)
-    (fp_text reference L3 (at 0 4.292601 90) (layer B.SilkS)
+    (fp_text reference L3 (at 0.254 2.286 90) (layer B.SilkS)
       (effects (font (thickness 0.3048)) (justify mirror))
     )
@@
     (at 166.37 102.235 90)
     (attr smd)
-    (fp_text reference C1 (at 0 -2.159 90) (layer F.SilkS)
+    (fp_text reference C1 (at -1.27 -2.032 90) (layer F.SilkS)
       (effects (font (size 1.016 1.00076) (thickness 0.15748)))
     )
@@
   )
   (module AK300-2 (layer Front-ext)
-    (at 168.275 130.175 90)
+    (at 168.021 130.175 90)
     (descr CONNECTOR)
     (tags CONNECTOR)
@@
     (descr "Diode 3 pas")
     (tags "DIODE DEV")
-    (fp_text reference D3 (at 0 0 180) (layer B.SilkS)
+    (fp_text reference D3 (at 0.889 0 180) (layer B.SilkS)
       (effects (font (size 1.016 1.016) (thickness 0.2032)) (justify mirror))
     )
@@
   )
   (module SIL-2 (layer Front-ext)
-    (at 177.8 127)
+    (at 177.8 127.762)
     (descr "Connecteurs 2 pins")
     (tags "CONN DEV")
@@
     (tags "FAIRCHILD'S TO-263AB/D2PAK PACKAGE DIMENSIONS")
     (attr smd)
-    (fp_text reference Q2 (at -6.8326 -0.12446 540) (layer B.SilkS)
-      (effects (font (size 1.27 1.27) (thickness 0.0889)) (justify mirror))
+    (fp_text reference Q2 (at -3.429 7.62 360) (layer B.SilkS)
+      (effects (font (size 1.27 1.27) (thickness 0.127)) (justify mirror))
     )
     (fp_text value 200V (at 1.905 7.62 360) (layer B.SilkS) hide
@@
   (gr_line (start 162.56 125.095) (end 162.56 133.985) (angle 90) (layer Edge.Cuts) (width 0.254))
   (gr_line (start 200.66 125.095) (end 200.66 133.985) (angle 90) (layer Edge.Cuts) (width 0.254))
-  (gr_text "5V\n\n        GND\n" (at 186.69 126.365) (layer B.SilkS)
+  (gr_text "5V\n\n        GND\n" (at 186.309 128.016) (layer B.SilkS)
     (effects (font (size 0.889 0.889) (thickness 0.127)) (justify mirror))
   )
-  (gr_text "BAT\n\n\nGND" (at 172.72 127.635) (layer B.SilkS)
+  (gr_text "BAT\n\n\nGND" (at 172.339 130.175) (layer B.SilkS)
     (effects (font (size 0.889 0.889) (thickness 0.127)) (justify mirror))
   )
-  (gr_text "Switching buck regulator aprox 80% eff\nInput 7V to 18V continious 3.5A max\npeak 100V for 40mS per ISO 7637-2\n\nOutput 4.XXV to 5.XXV \nat 3A with XX Vripple " (at 200.025 133.35 270) (layer B.SilkS)
+  (gr_text "Switching buck regulator aprox 80% eff\nInput 7V to 18V continious 3.5A max\npeak 100V for 40mS per ISO 7637-2\n\nOutput 4.XXV to 5.XXV \nat 3A with XX Vripple " (at 195.453 133.223 270) (layer B.SilkS)
     (effects (font (size 1.016 1.016) (thickness 0.127)) (justify left mirror))
   )
-  (gr_text "for rusEFI\nhttps://sourceforge.net/p/rusefi/" (at 194.31 108.585) (layer B.SilkS)
+  (gr_text "for rusEFI\nhttps://sourceforge.net/p/rusefi/" (at 193.675 113.157) (layer B.SilkS)
     (effects (font (size 1.016 1.016) (thickness 0.127)) (justify left mirror))
   )
-  (gr_text R0.3 (at 168.275 102.235) (layer B.SilkS)
+  (gr_text R0.4 (at 189.865 110.363) (layer B.SilkS)
     (effects (font (size 1.016 1.016) (thickness 0.127)) (justify mirror))
   )
@@
     (effects (font (size 1.016 1.016) (thickness 0.127)) (justify mirror))
   )
-  (gr_text "TEST POINT\n        P2\n\n\n" (at 187.96 102.235) (layer B.SilkS)
+  (gr_text "TEST POINT\n        P2\n\n\n" (at 187.96 104.394) (layer B.SilkS)
     (effects (font (size 1.016 1.016) (thickness 0.127)) (justify mirror))
   )
@@
   (segment (start 186.69 96.52) (end 188.595 98.425) (width 1.38176) (layer Front-ext) (net 3))
   (segment (start 188.595 98.425) (end 188.595 100.965) (width 1.38176) (layer Front-ext) (net 3))
-  (segment (start 168.275 101.06914) (end 167.36314 101.06914) (width 0.254) (layer Back-ext) (net 4))
-  (segment (start 167.36314 101.06914) (end 163.576 97.282) (width 0.254) (layer Back-ext) (net 4))
+  (segment (start 168.275 101.06914) (end 167.36314 101.06914) (width 1.38176) (layer Back-ext) (net 4))
+  (segment (start 167.36314 101.06914) (end 165.354 99.06) (width 1.38176) (layer Back-ext) (net 4))
+  (segment (start 165.354 99.06) (end 163.576 99.06) (width 1.38176) (layer Back-ext) (net 4))
+  (segment (start 167.36314 101.06914) (end 163.576 97.282) (width 1.38176) (layer Back-ext) (net 4))
   (segment (start 166.37 106.63428) (end 166.37 106.045) (width 1.38176) (layer Front-ext) (net 4))
   (segment (start 166.37 106.045) (end 168.275 104.14) (width 1.38176) (layer Front-ext) (net 4))
@@
   (segment (start 173.30928 106.63428) (end 166.37 106.63428) (width 1.38176) (layer Front-ext) (net 4))
   (segment (start 174.3964 107.7214) (end 173.30928 106.63428) (width 1.38176) (layer Front-ext) (net 4))
-  (segment (start 184.62498 123.14936) (end 186.41314 123.14936) (width 1.38176) (layer Back-ext) (net 5))
-  (segment (start 186.41314 123.14936) (end 187.96 121.6025) (width 1.38176) (layer Back-ext) (net 5))
-  (segment (start 179.07 127) (end 180.77434 127) (width 1.38176) (layer Back-ext) (net 5))
-  (segment (start 180.77434 127) (end 184.62498 123.14936) (width 1.38176) (layer Back-ext) (net 5))
-  (segment (start 168.275 127.6858) (end 175.8442 127.6858) (width 1.38176) (layer Front-ext) (net 6))
-  (segment (start 175.8442 127.6858) (end 176.53 127) (width 1.38176) (layer Front-ext) (net 6))
-  (segment (start 184.62498 118.15064) (end 186.41314 118.15064) (width 1.38176) (layer Back-ext) (net 7))
-  (segment (start 186.41314 118.15064) (end 187.96 119.6975) (width 1.38176) (layer Back-ext) (net 7))
+  (segment (start 187.96 121.6025) (end 187.8965 121.6025) (width 0.254) (layer Back-ext) (net 5))
+  (segment (start 187.8965 121.6025) (end 186.34964 123.14936) (width 0.254) (layer Back-ext) (net 5))
+  (segment (start 186.34964 123.14936) (end 184.62498 123.14936) (width 0.254) (layer Back-ext) (net 5))
+  (segment (start 180.01234 127.762) (end 184.62498 123.14936) (width 1.38176) (layer Back-ext) (net 5))
+  (segment (start 179.07 127.762) (end 180.01234 127.762) (width 1.38176) (layer Back-ext) (net 5))
+  (segment (start 176.53 127.762) (end 168.0972 127.762) (width 1.38176) (layer Back-ext) (net 6))
+  (segment (start 168.0972 127.762) (end 168.021 127.6858) (width 1.38176) (layer Back-ext) (net 6))
+  (segment (start 184.62498 118.15064) (end 186.73064 118.15064) (width 0.254) (layer Back-ext) (net 7))
+  (segment (start 186.73064 118.15064) (end 187.96 119.38) (width 0.254) (layer Back-ext) (net 7))
+  (segment (start 187.96 119.38) (end 187.96 119.6975) (width 0.254) (layer Back-ext) (net 7))
   (segment (start 184.62498 118.15064) (end 184.19064 118.15064) (width 1.38176) (layer Back-ext) (net 7))
   (segment (start 164.465 114.3) (end 163.83 113.665) (width 1.38176) (layer Back-ext) (net 7))

Commit message: auto-sync
Parts:
- moved R3 8.98 mm to (181.6, 114.3)
Connections:
- Q2 pad 2: /Vs2 -> /Vf
- Q2 pad 3: /Vf -> /Vs2
Routing:
- net /Vs2: track 8.95 -> 23.8 mm
- net /Vf: track 11.4 -> 18.2 mm
- net /Vs1: track 26.8 -> 25.7 mm
- net GND: vias 21 -> 20
Other:
- net class 5A EXT 200V: clearance 1.016 -> 0.762
- board text added: "R0.5"
- board text added: "https://sourceforge.net/p/rusefi/"
- board text removed: "R0.4"
- board text removed: "for rusEFI https://sourceforge.net/p/rusefi/"
Changed lines of the file:
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@@
-(kicad_pcb (version 4) (host pcbnew 4.0.1-stable)
+(kicad_pcb (version 4) (host pcbnew 4.0.5)
   (general
     (links 40)
     (no_connects 0)
-    (area 159.457572 92.71 212.697787 141.986)
+    (area 159.838572 92.71 212.507287 142.0241)
     (thickness 1.6002)
     (drawings 19)
-    (tracks 125)
+    (tracks 126)
     (zones 0)
     (modules 24)
@@
   (title_block
     (title "PWR buck 12V switcher regulator")
-    (rev "R 0.4")
+    (date 2017-02-12)
+    (rev "R 0.5")
     (company https://sourceforge.net/p/rusefi/)
   )
@@
   )
   (setup
-    (last_trace_width 0.254)
+    (last_trace_width 0.2032)
     (user_trace_width 0.254)
     (user_trace_width 0.39116)
@@
     (uvia_dia 0.762)
     (uvia_drill 0.254)
+    (add_net /Vs1)
   )
   (net_class "1A INT" ""
@@
     (add_net /OUT)
     (add_net /VBAT)
-    (add_net /Vs1)
     (add_net /Vs2)
     (add_net GND)
@@
   )
   (net_class "5A EXT 200V" ""
-    (clearance 1.016)
+    (clearance 0.762)
     (trace_width 1.38176)
     (via_dia 1.651)
@@
   )
   (module SM0805 (layer Back-ext)
-    (at 187.96 120.65 90)
+    (at 181.61 114.3 90)
     (attr smd)
     (fp_text reference R3 (at 0 0 360) (layer B.SilkS)
@@
     (fp_line (start 3.29946 -7.0993) (end 3.29946 -4.49834) (layer B.SilkS) (width 0.127))
     (pad 2 smd rect (at 0 0 270) (size 9.99998 8.99922) (layers Back-ext B.Paste B.Mask)
-      (net 8 /Vs2))
+      (net 5 /Vf))
     (pad 1 smd rect (at -2.49936 -9.99998 270) (size 1.4986 3.99796) (layers Back-ext B.Paste B.Mask)
       (net 7 /Vs1))
     (pad 3 smd rect (at 2.49936 -9.99998 270) (size 1.4986 3.99796) (layers Back-ext B.Paste B.Mask)
-      (net 5 /Vf))
+      (net 8 /Vs2))
   )
   (gr_line (start 200.66 110.617) (end 200.66 110.49) (angle 90) (layer F.SilkS) (width 0.254))
@@
     (effects (font (size 0.889 0.889) (thickness 0.127)) (justify mirror))
   )
-  (gr_text "Switching buck regulator aprox 80% eff\nInput 7V to 18V continious 3.5A max\npeak 100V for 40mS per ISO 7637-2\n\nOutput 4.XXV to 5.XXV \nat 3A with XX Vripple " (at 195.453 133.223 270) (layer B.SilkS)
+  (gr_text "Switching buck regulator aprox 80% eff\nInput 7V to 18V continious 3.5A max\npeak 100V for 40mS per ISO 7637-2\n\nOutput 4.XXV to 5.XXV \nat 3A with XX Vripple " (at 195.453 127.381 270) (layer B.SilkS)
     (effects (font (size 1.016 1.016) (thickness 0.127)) (justify left mirror))
   )
-  (gr_text "for rusEFI\nhttps://sourceforge.net/p/rusefi/" (at 193.675 113.157) (layer B.SilkS)
+  (gr_text https://sourceforge.net/p/rusefi/ (at 189.357 125.603 270) (layer B.SilkS)
     (effects (font (size 1.016 1.016) (thickness 0.127)) (justify left mirror))
   )
-  (gr_text R0.4 (at 189.865 110.363) (layer B.SilkS)
+  (gr_text R0.5 (at 186.182 113.411 270) (layer B.SilkS)
     (effects (font (size 1.016 1.016) (thickness 0.127)) (justify mirror))
   )
@@
     (effects (font (size 1.016 1.016) (thickness 0.127)) (justify mirror))
   )
-  (gr_text "TEST POINT\n        P2\n\n\n" (at 187.96 104.394) (layer B.SilkS)
+  (gr_text "TEST\nPOINT\n P2\n\n\n" (at 185.293 103.505) (layer B.SilkS)
     (effects (font (size 1.016 1.016) (thickness 0.127)) (justify mirror))
   )
@@
   (segment (start 173.30928 106.63428) (end 166.37 106.63428) (width 1.38176) (layer Front-ext) (net 4))
   (segment (start 174.3964 107.7214) (end 173.30928 106.63428) (width 1.38176) (layer Front-ext) (net 4))
-  (segment (start 187.96 121.6025) (end 187.8965 121.6025) (width 0.254) (layer Back-ext) (net 5))
-  (segment (start 187.8965 121.6025) (end 186.34964 123.14936) (width 0.254) (layer Back-ext) (net 5))
-  (segment (start 186.34964 123.14936) (end 184.62498 123.14936) (width 0.254) (layer Back-ext) (net 5))
-  (segment (start 180.01234 127.762) (end 184.62498 123.14936) (width 1.38176) (layer Back-ext) (net 5))
-  (segment (start 179.07 127.762) (end 180.01234 127.762) (width 1.38176) (layer Back-ext) (net 5))
+  (segment (start 181.61 115.2525) (end 180.0225 115.2525) (width 1.38176) (layer Back-ext) (net 5))
+  (segment (start 180.0225 115.2525) (end 174.625 120.65) (width 1.38176) (layer Back-ext) (net 5))
+  (segment (start 179.07 127.762) (end 179.07 125.095) (width 1.38176) (layer Back-ext) (net 5))
+  (segment (start 179.07 125.095) (end 174.625 120.65) (width 1.38176) (layer Back-ext) (net 5))
   (segment (start 176.53 127.762) (end 168.0972 127.762) (width 1.38176) (layer Back-ext) (net 6))
   (segment (start 168.0972 127.762) (end 168.021 127.6858) (width 1.38176) (layer Back-ext) (net 6))
-  (segment (start 184.62498 118.15064) (end 186.73064 118.15064) (width 0.254) (layer Back-ext) (net 7))
-  (segment (start 186.73064 118.15064) (end 187.96 119.38) (width 0.254) (layer Back-ext) (net 7))
-  (segment (start 187.96 119.38) (end 187.96 119.6975) (width 0.254) (layer Back-ext) (net 7))
+  (segment (start 184.62498 118.15064) (end 184.62498 114.13998) (width 0.254) (layer Back-ext) (net 7))
+  (segment (start 183.8325 113.3475) (end 181.61 113.3475) (width 0.254) (layer Back-ext) (net 7))
+  (segment (start 184.62498 114.13998) (end 183.8325 113.3475) (width 0.254) (layer Back-ext) (net 7))
+  (segment (start 181.61 113.3475) (end 164.1475 113.3475) (width 0.254) (layer Back-ext) (net 7))
+  (segment (start 164.1475 113.3475) (end 163.83 113.665) (width 0.254) (layer Back-ext) (net 7))
   (segment (start 184.62498 118.15064) (end 184.19064 118.15064) (width 1.38176) (layer Back-ext) (net 7))
-  (segment (start 164.465 114.3) (end 163.83 113.665) (width 1.38176) (layer Back-ext) (net 7))
-  (segment (start 180.34 114.3) (end 164.465 114.3) (width 1.38176) (layer Back-ext) (net 7))
-  (segment (start 184.19064 118.15064) (end 180.34 114.3) (width 1.38176) (layer Back-ext) (net 7))
-  (segment (start 174.625 120.65) (end 169.545 120.65) (width 1.38176) (layer Back-ext) (net 8))
-  (segment (start 168.275 119.38) (end 168.275 117.30482) (width 1.38176) (layer Front-ext) (net 8))
-  (via (at 168.275 119.38) (size 1.651) (layers Front-ext Back-ext) (net 8))
-  (segment (start 169.545 120.65) (end 168.275 119.38) (width 1.38176) (layer Back-ext) (net 8))
+  (segment (start 184.62498 123.14936) (end 184.62498 123.35002) (width 1.38176) (layer Back-ext) (net 8))
+  (segment (start 184.62498 123.35002) (end 182.88 125.095) (width 1.38176) (layer Back-ext) (net 8))
+  (segment (start 168.275 120.015) (end 168.275 117.30482) (width 1.38176) (layer Front-ext) (net 8))
+  (segment (start 170.815 122.555) (end 168.275 120.015) (width 1.38176) (layer Front-ext) (net 8))
+  (segment (start 180.34 122.555) (end 170.815 122.555) (width 1.38176) (layer Front-ext) (net 8))
+  (segment (start 182.88 125.095) (end 180.34 122.555) (width 1.38176) (layer Front-ext) (net 8))
+  (via (at 182.88 125.095) (size 1.651) (drill 1.143) (layers Front-ext Back-ext) (net 8))
+  (segment (start 186.34964 123.14936) (end 184.62498 123.14936) (width 0.254) (layer Back-ext) (net 8))
   (segment (start 172.085 108.2675) (end 171.0055 108.2675) (width 0.254) (layer Front-ext) (net 9))
   (via (at 170.815 108.077) (size 1.016) (drill 0.508) (layers Front-ext Back-ext) (net 9))
@@
   (segment (start 196.215 104.521) (end 194.945 103.251) (width 1.38176) (layer Front-ext) (net 9))
   (segment (start 183.69026 109.22) (end 182.245 110.66526) (width 1.38176) (layer Front-ext) (net 9))
-  (via (at 182.245 111.76) (size 1.651) (layers Front-ext Back-ext) (net 9))
   (segment (start 182.245 110.66526) (end 182.245 111.76) (width 1.38176) (layer Front-ext) (net 9))
   (segment (start 177.8 109.22) (end 177.8 111.76) (width 1.38176) (layer Front-ext) (net 9))
