File: hardware/NUCLEO144_wing/NUCLEO144_wing.kicad_pcb (KiCad board)
At the start: 4 copper layers, 11 x 9 mm, 0 parts

Commit message: p
Other:
- board outline removed
- board text removed: "1"
- board text removed: "2"
Changed lines of the file:
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@@
 (kicad_pcb (version 4) (host pcbnew 4.0.7)
   (general
-    (links 3)
-    (no_connects 1)
-    (area 66.040002 20.32 284.480001 227.749101)
+    (links 0)
+    (no_connects 0)
+    (area 66.040002 20.32 284.480001 216.2048)
     (thickness 1.6)
-    (drawings 18)
+    (drawings 9)
     (tracks 0)
     (zones 0)
@@
   (page B)
   (title_block
-    (title Frankenso)
-    (date 2018-02-24)
-    (rev R0.5.3)
+    (title nucleo144_wing)
+    (date 2019-02-24)
+    (rev R0.1)
     (company http://rusefi.com/)
   )
@@
     (uvia_dia 0.508)
     (uvia_drill 0.127)
-    (add_net /HD44780_CS)
-    (add_net /HD44780_D4)
-    (add_net /HD44780_D5)
-    (add_net /HD44780_D6)
-    (add_net /HD44780_D7)
-    (add_net /HD44780_RS)
-    (add_net /HD44780_VCC)
-    (add_net /HD44780_VLCD)
-    (add_net GND)
   )
   (net_class "1A external" ""
@@
     (effects (font (size 1.016 1.016) (thickness 0.127)) (justify left))
   )
-  (gr_text "  2 " (at 109.855 188.976) (layer GND)
-    (effects (font (size 1.016 1.016) (thickness 0.127)) (justify left))
-  )
-  (gr_text " 1  " (at 109.855 188.976) (layer PWR)
-    (effects (font (size 1.016 1.016) (thickness 0.127)) (justify left))
-  )
   (gr_text "0   " (at 109.855 188.976) (layer F.Cu)
     (effects (font (size 1.016 1.016) (thickness 0.127)) (justify left))
@@
   (target plus (at 107.95 203.2) (size 0.005) (width 0.127) (layer Edge.Cuts))
   (target plus (at 107.95 203.2) (size 0.005) (width 0.127) (layer Edge.Cuts))
-  (dimension 154.1272 (width 0.127) (layer Dwgs.User)
-    (gr_text "6.0680 in" (at 185.42 226.06) (layer Dwgs.User)
-      (effects (font (size 2.032 2.032) (thickness 0.127)))
-    )
-    (feature1 (pts (xy 262.1788 188.214) (xy 262.178799 223.799403)))
-    (feature2 (pts (xy 108.0516 188.214) (xy 108.051599 223.799403)))
-    (crossbar (pts (xy 108.051599 222.783403) (xy 262.178799 222.783403)))
-    (arrow1a (pts (xy 262.178799 222.783403) (xy 261.052296 223.369823)))
-    (arrow1b (pts (xy 262.178799 222.783403) (xy 261.052296 222.196983)))
-    (arrow2a (pts (xy 108.051599 222.783403) (xy 109.178102 223.369823)))
-    (arrow2b (pts (xy 108.051599 222.783403) (xy 109.178102 222.196983)))
-  )
-  (gr_line (start 118.872 189.992) (end 118.872 179.578) (angle 90) (layer Dwgs.User) (width 0.381))
-  (gr_line (start 131.826 189.992) (end 118.872 189.992) (angle 90) (layer Dwgs.User) (width 0.381))
-  (dimension 138.811 (width 0.3048) (layer Dwgs.User)
-    (gr_text "5.4650 in" (at 97.0534 120.5865 90) (layer Dwgs.User)
-      (effects (font (size 2.032 1.524) (thickness 0.3048)))
-    )
-    (feature1 (pts (xy 110.998 51.181) (xy 95.4278 51.181)))
-    (feature2 (pts (xy 110.998 189.992) (xy 95.4278 189.992)))
-    (crossbar (pts (xy 98.679 189.992) (xy 98.679 51.181)))
-    (arrow1a (pts (xy 98.679 51.181) (xy 99.26542 52.307503)))
-    (arrow1b (pts (xy 98.679 51.181) (xy 98.09258 52.307503)))
-    (arrow2a (pts (xy 98.679 189.992) (xy 99.26542 188.865497)))
-    (arrow2b (pts (xy 98.679 189.992) (xy 98.09258 188.865497)))
-  )
-  (gr_line (start 113.04904 189.95634) (end 111.046 189.95634) (angle 90) (layer Edge.Cuts) (width 0.127))
-  (gr_arc (start 113.04904 195.9609) (end 119.0536 195.9609) (angle -90) (layer Edge.Cuts) (width 0.127))
-  (gr_arc (start 111.046 186.95406) (end 108.04372 186.95406) (angle -90) (layer Edge.Cuts) (width 0.127))
   (zone (net 1) (net_name GND) (layer F.Cu) (hatch edge 0.508)
     (connect_pads (clearance 0.254))
     (min_thickness 0.254)
-    (fill yes (arc_segments 16) (thermal_gap 0.254) (thermal_bridge_width 0.508))
+    (fill (arc_segments 16) (thermal_gap 0.254) (thermal_bridge_width 0.508))
     (polygon
       (pts
         (xy 276.86 208.28) (xy 104.14 208.28) (xy 104.14 27.94) (xy 276.86 27.94)
-      )
-    )
-    (polygon
-      (pts        (xy 185.42 66.04) (xy 185.42 50.8) (xy 172.72 50.8) (xy 172.72 66.04)
-      )
-    )
-    (polygon
-      (pts        (xy 262.89 192.405) (xy 262.89 183.515) (xy 244.475 183.515) (xy 244.475 206.375)
-      )
-    )
-    (polygon
-      (pts        (xy 107.315 125.095) (xy 118.11 125.095) (xy 118.11 148.59) (xy 107.315 148.59)
-      )
-    )
-    (polygon
-      (pts        (xy 109.855 68.58) (xy 110.744 68.58) (xy 111.125 68.961) (xy 111.125 69.469) (xy 112.522 69.469)
-        (xy 113.03 68.961) (xy 114.3 68.961) (xy 114.3 71.755) (xy 116.713 71.755) (xy 116.713 69.469)
-        (xy 116.459 69.215) (xy 116.713 68.961) (xy 117.094 68.961) (xy 117.348 69.215) (xy 117.348 69.977)
-        (xy 122.428 69.977) (xy 123.571 71.12) (xy 126.873 71.12) (xy 126.873 68.326) (xy 127.508 68.326)
-        (xy 127.508 60.071) (xy 126.238 58.801) (xy 117.221 58.801) (xy 117.221 61.087) (xy 116.205 62.103)
-        (xy 116.205 62.865) (xy 114.681 64.389) (xy 113.157 65.913) (xy 109.855 65.913)
       )
     )
@@
     (connect_pads (clearance 0.254))
     (min_thickness 0.254)
-    (fill yes (arc_segments 16) (thermal_gap 0.254) (thermal_bridge_width 0.508))
+    (fill (arc_segments 16) (thermal_gap 0.254) (thermal_bridge_width 0.508))
     (polygon
       (pts
         (xy 279.4 210.82) (xy 101.6 210.82) (xy 101.6 25.4) (xy 279.4 25.4)
-      )
-    )
-    (polygon
-      (pts        (xy 244.475 183.515) (xy 244.475 207.01) (xy 263.525 193.04) (xy 263.525 183.515)
-      )
-    )
-    (polygon
-      (pts        (xy 102.87 125.095) (xy 102.87 148.59) (xy 118.11 148.59) (xy 118.11 125.095)
-      )
-    )
-    (polygon
-      (pts        (xy 172.72 50.8) (xy 172.72 66.04) (xy 185.42 66.04) (xy 187.96 59.69) (xy 185.42 50.8)
       )
     )
@@
     (connect_pads (clearance 0.2159))
     (min_thickness 0.2159)
-    (fill yes (arc_segments 16) (thermal_gap 0.508) (thermal_bridge_width 0.508) (smoothing fillet) (radius 0.508))
+    (fill (arc_segments 16) (thermal_gap 0.508) (thermal_bridge_width 0.508) (smoothing fillet) (radius 0.508))
     (polygon
       (pts
         (xy 281.94 213.36) (xy 99.06 213.36) (xy 99.06 22.86) (xy 281.94 22.86)
-      )
-    )
-    (polygon
-      (pts        (xy 244.475 183.515) (xy 244.475 207.645) (xy 264.16 193.675) (xy 264.16 183.515)
-      )
-    )
-    (polygon
-      (pts        (xy 102.235 125.095) (xy 102.235 148.59) (xy 118.11 148.59) (xy 118.11 125.095)
-      )
-    )
-    (polygon
-      (pts        (xy 106.045 39.37) (xy 106.045 69.215) (xy 129.54 69.215) (xy 129.54 52.07) (xy 136.525 52.07)
-        (xy 136.525 39.37)
-      )
-    )
-    (polygon
-      (pts        (xy 172.72 50.8) (xy 172.72 66.04) (xy 185.42 66.04) (xy 185.42 50.8)
       )
     )
@@
     (connect_pads (clearance 0.2159))
     (min_thickness 0.2159)
-    (fill yes (arc_segments 16) (thermal_gap 0.508) (thermal_bridge_width 0.508) (smoothing fillet) (radius 0.508))
+    (fill (arc_segments 16) (thermal_gap 0.508) (thermal_bridge_width 0.508) (smoothing fillet) (radius 0.508))
     (polygon
       (pts
@@
       )
     )
-    (polygon
-      (pts        (xy 244.475 183.515) (xy 244.475 208.28) (xy 264.795 194.31) (xy 264.795 183.515)
-      )
-    )
-    (polygon
-      (pts        (xy 98.425 125.095) (xy 98.425 148.59) (xy 118.11 148.59) (xy 118.11 125.095)
-      )
-    )
-    (polygon
-      (pts        (xy 105.41 38.735) (xy 105.41 69.215) (xy 129.54 69.215) (xy 129.54 52.07) (xy 136.525 52.07)
-        (xy 136.525 38.735)
-      )
-    )
-    (polygon
-      (pts        (xy 172.72 50.8) (xy 172.72 66.04) (xy 185.42 66.04) (xy 185.42 50.8)
-      )
-    )

Commit message: p
Parts:
- added U1: NUCLEO144-F429ZI, rusEFI_LIB:ST_Morpho_Connector_144_STLink, F.Cu at (97.8, 57.1)
- added U2: NUCLEO144-F429ZI, rusEFI_LIB:ST_Morpho_Connector_144_STLink, F.Cu at (237.5, 57.1)
Routing:
- removed copper zone on PWR, net /5V
- removed copper zone on GND, net GND
Other:
- board outline added: 100 x 100 mm
- copper layers 4 -> 2
- board text added: "2 layer board stackup is as follows: 0 is top min 1 oz copper (1.4 mil) min 47 mil core FR4 3 is bottom min 1 oz copper (1.4 mil)"
- board text removed: "4 layer board stackup is as follows: 0 is top min 1 oz copper (1.4 mil) min 6.7 mil prepreg FR4 1 is GND min 0.5 oz copper (0.7 mil) min 47 mil core FR4 2 is PWR min 0.5 oz copper (0.7 mil) min 6.7 mil prepreg FR4 3 is bottom min 1 oz copper (1.4 mil)"

Commit message: p
Parts:
- added J1: Conn_02x36_Top_Bottom, Pin_Headers:Pin_Header_Straight_2x36_Pitch2.54mm, F.Cu at (234.9, 54.6)
- added J2: Conn_02x36_Top_Bottom, Pin_Headers:Pin_Header_Straight_2x36_Pitch2.54mm, F.Cu at (245.1, 54.6)
- moved U2 54.6 mm to (292.1, 57.1)
- moved U1 41.4 mm to (58.4, 44.5)
Routing:
- net (no net): track 0.00 -> 89.7 mm
- net Net-(J1-Pad1): track 0.00 -> 13.0 mm
- net Net-(J1-Pad2): track 0.00 -> 13.0 mm
- net Net-(J1-Pad70): track 0.00 -> 11.2 mm
- net Net-(J1-Pad68): track 0.00 -> 11.2 mm
- net Net-(J1-Pad62): track 0.00 -> 11.2 mm
- net Net-(J1-Pad60): track 0.00 -> 11.2 mm
- net Net-(J1-Pad58): track 0.00 -> 11.2 mm
- net Net-(J1-Pad54): track 0.00 -> 11.2 mm
- net Net-(J1-Pad5): track 0.00 -> 11.2 mm
- net Net-(J1-Pad40): track 0.00 -> 11.2 mm
- net Net-(J1-Pad36): track 0.00 -> 11.2 mm
- net Net-(J1-Pad3): track 0.00 -> 11.2 mm
- net Net-(J1-Pad26): track 0.00 -> 11.2 mm
- net Net-(J1-Pad22): track 0.00 -> 11.2 mm
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Other:
- net class Default: clearance 0.1524 -> 0.254; trace_width 0.1524 -> 0.254
- rule trace_clearance: 0.1524 -> 0.254
- board text added: "C11"

Commit message: p
Parts:
- added J3: Conn_02x36_Top_Bottom, Pin_Headers:Pin_Header_Straight_2x36_Pitch2.54mm, F.Cu at (152.4, 54.6)
- added J4: Conn_02x36_Top_Bottom, Pin_Headers:Pin_Header_Straight_2x36_Pitch2.54mm, F.Cu at (162.6, 54.6)
Connections:
- J2 pad 23: Net-(J2-Pad23) -> Net-(J1-Pad23)
- J2 pad 25: Net-(J2-Pad25) -> Net-(J1-Pad25)
- J2 pad 27: Net-(J2-Pad27) -> Net-(J1-Pad27)
- J2 pad 29: Net-(J2-Pad29) -> Net-(J1-Pad29)
- J2 pad 31: Net-(J2-Pad31) -> Net-(J1-Pad31)
- J2 pad 33: Net-(J2-Pad33) -> Net-(J1-Pad33)
- J2 pad 35: Net-(J2-Pad35) -> Net-(J1-Pad35)
- J2 pad 37: Net-(J2-Pad37) -> Net-(J1-Pad37)
- J2 pad 39: Net-(J2-Pad39) -> Net-(J1-Pad39)
- J2 pad 41: Net-(J2-Pad41) -> Net-(J1-Pad41)
- J2 pad 43: Net-(J2-Pad43) -> Net-(J1-Pad43)
- J2 pad 45: Net-(J2-Pad45) -> Net-(J1-Pad45)
- J2 pad 47: Net-(J2-Pad47) -> Net-(J1-Pad47)
- J2 pad 49: Net-(J2-Pad49) -> Net-(J1-Pad49)
- J2 pad 51: Net-(J2-Pad51) -> Net-(J1-Pad51)
- J2 pad 53: Net-(J2-Pad53) -> Net-(J1-Pad53)
- J2 pad 55: Net-(J2-Pad55) -> Net-(J1-Pad55)
- J2 pad 57: Net-(J2-Pad57) -> Net-(J1-Pad57)
- J2 pad 59: Net-(J2-Pad59) -> Net-(J1-Pad59)
- J2 pad 61: Net-(J2-Pad61) -> Net-(J1-Pad61)
- J2 pad 63: Net-(J2-Pad63) -> Net-(J1-Pad63)
- J2 pad 65: Net-(J2-Pad65) -> Net-(J1-Pad65)
- J2 pad 67: Net-(J2-Pad67) -> Net-(J1-Pad67)
- J2 pad 69: Net-(J2-Pad69) -> Net-(J1-Pad69)
- J2 pad 71: Net-(J2-Pad71) -> Net-(J1-Pad71)
Routing:
- net (no net): track 89.7 -> 44.8 mm
- net Net-(J1-Pad69): track 0.00 -> 11.2 mm
- net Net-(J1-Pad67): track 0.00 -> 11.2 mm
- net Net-(J1-Pad59): track 0.00 -> 11.2 mm
- net Net-(J1-Pad57): track 0.00 -> 11.2 mm
- net Net-(J1-Pad53): track 0.00 -> 11.2 mm
- net Net-(J1-Pad39): track 0.00 -> 11.2 mm
- net Net-(J1-Pad35): track 0.00 -> 11.2 mm
- net Net-(J1-Pad25): track 0.00 -> 11.2 mm
- net Net-(J1-Pad21): track 0.00 -> 11.2 mm
- net Net-(J1-Pad17): track 0.00 -> 11.2 mm
- net Net-(J1-Pad61): track 0.00 -> 11.2 mm
- net Net-(J3-Pad70): track 0.00 -> 11.2 mm
- net Net-(J3-Pad69): track 0.00 -> 11.2 mm
- net Net-(J3-Pad68): track 0.00 -> 11.2 mm
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Other:
- board text added: "A13"
- board text added: "A14"
- board text added: "A15"
- board text added: "B7"
- board text added: "BT0"
- board text added: "C10"
- board text added: "C12"
- board text added: "C13"
- board text added: "C14"
- board text added: "C15"
- board text added: "C2"
- board text added: "C3"
- board text added: "D0"
- board text added: "D1"
- board text added: "D2"
- board text added: "D4"
- board text added: "D5"
- board text added: "D6"
- board text added: "D7"
- board text added: "D9"
- board text added: "E1"
- board text added: "E3"
- board text added: "F0"
- board text added: "F1"
- board text added: "F6"
- board text added: "F7"
- board text added: "G0"
- board text added: "G12"
- board text added: "G9"
- board text added: "GND"
- board text added: "H0"
- board text added: "H1"
- board text added: "N144 Wing 0.1"
- board text added: "NC"
- board text added: "VBAT"
- board text added: "VDD"
- board text added: "X"
- board text added: "XX"

Commit message: silk phase #1
Routing:
- net (no net): track 44.8 -> 0.00 mm
Other:
- board text added: "3V3"
- board text added: "5V"
- board text added: "A0"
- board text added: "A1"
- board text added: "A10"
- board text added: "A11"
- board text added: "A12"
- board text added: "A2"
- board text added: "A3"
- board text added: "A4"
- board text added: "A5"
- board text added: "A6"
- board text added: "A7"
- board text added: "A8"
- board text added: "A9"
- board text added: "AGND"
- board text added: "AVDD"
- board text added: "B0"
- board text added: "B1"
- board text added: "B10"
- board text added: "B11"
- board text added: "B12"
- board text added: "B13"
- board text added: "B14"
- board text added: "B15"
- board text added: "B2"
- board text added: "B3"
- board text added: "B4"
- board text added: "B5"
- board text added: "B6"
- board text added: "B8"
- board text added: "B9"
- board text added: "C0"
- board text added: "C1"
- board text added: "C4"
- board text added: "C5"
- board text added: "C6"
- board text added: "C7"
- board text added: "C8"
- board text added: "C9"
- board text added: "D10"
- board text added: "D11"
- board text added: "D12"
- board text added: "D13"
- board text added: "D14"
- board text added: "D15"
- board text added: "D3"
- board text added: "D8"
- board text added: "E0"
- board text added: "E10"
- board text added: "E11"
- board text added: "E12"
- board text added: "E13"
- board text added: "E14"
- board text added: "E15"
- board text added: "E2"
- board text added: "E4"
- board text added: "E5"
- board text added: "E5V"
- board text added: "E6"
- board text added: "E7"
- board text added: "E8"
- board text added: "E9"
- board text added: "F10"
- board text added: "F11"
- board text added: "F12"
- board text added: "F13"
- board text added: "F14"
- board text added: "F15"
- board text added: "F2"
- board text added: "F3"
- board text added: "F4"
- board text added: "F5"
- board text added: "F8"
- board text added: "F9"
- board text added: "G1"
- board text added: "G10"
- board text added: "G11"
- board text added: "G13"
- board text added: "G14"
- board text added: "G15"
- board text added: "G2"
- board text added: "G3"
- board text added: "G4"
- board text added: "G5"
- board text added: "G6"
- board text added: "G7"
- board text added: "G8"
- board text added: "NRST"
- board text added: "U5V"
- board text added: "VIN"
- board text added: "rusEfi.com"
- board text removed: "X"
- board text removed: "XX"

Commit message: p
Parts:
- added REF**: Pin_Header_Straight_1x24_Pitch2.54mm, Pin_Headers:Pin_Header_Straight_1x24_Pitch2.54mm, F.Cu at (169.4, 154.9)
- moved J1 1.02 mm to (236.0, 54.6)
- moved J3 1.02 mm to (151.4, 54.6)
- moved J2 1.02 mm to (246.1, 54.6)
- moved J4 1.02 mm to (161.5, 54.6)

Commit message: p
Parts:
- added REF**: rusEfi_4x39_Pitch2.54mm, rusEFI_local:rusEfi_4x39_Pitch2.54mm, F.Cu at (173.0, 50.3)
- added REF**: rusEfi_4x39_Pitch2.54mm, rusEFI_local:rusEfi_4x39_Pitch2.54mm, F.Cu at (194.3, 53.6)
