File: hardware/176122-6-connector/176122-6.kicad_pcb (KiCad board)
At the start: 2 copper layers, 137.2 x 33.2 mm, 43 parts, among them P1 CONN_3, P10 CONN_1, P11 CONN_1, P12 CONN_1, P13 CONN_3, P14 CONN_3, P15 CONN_1, P16 CONN_1, P17 CONN_1, P18 CONN_1, P19 CONN_1, P2 CONN_3, P20 CONN_1, P21 CONN_1, P22 CONN_1, P23 CONN_1, P24 CONN_1, P25 0176122-06, P26 CONN_8, P27 CONN_8, P28 CONN_8, P29 CONN_8, P3 CONN_1, P30 CONN_8, P31 CONN_8, P32 CONN_8, P33 CONN_8, P34 CONN_8, P35 CONN_8, P36 CONN_8, P37 CONN_8, P38 CONN_1, P39 CONN_1, P4 CONN_1, P40 CONN_1, P41 CONN_1, P5 CONN_1, P6 CONN_1, P7 CONN_1, P8 CONN_1, P9 CONN_1

Commit message: Updated to KC5
Parts:
- P1, P13, P14, P2: footprint SIL-3 -> Connector_PinHeader_2.54mm:PinHeader_1x03_P2.54mm_Vertical
- P10, P11, P12, P15, P16, P17, P18, P19, P20, P21, P22, P23, P24, P3, P38, P39, P4, P40, P41, P5, P6, P7, P8, P9: footprint SIL-1 -> Connector_PinHeader_2.54mm:PinHeader_1x01_P2.54mm_Vertical
- P25: footprint 176122-6 -> 0176122-06:176122-6
- P26, P27, P28, P29, P30, P31, P32, P33, P34, P35, P36, P37: footprint SIL-8 -> Connector_PinHeader_2.54mm:PinHeader_1x08_P2.54mm_Vertical
- moved P31 11.5 mm to (95.5, 62.2), turned to 270 degrees
- moved P37 11.5 mm to (95.5, 69.6), turned to 270 degrees
- moved P30 11.5 mm to (95.5, 64.8), turned to 270 degrees
- moved P36 11.5 mm to (95.5, 72.1), turned to 270 degrees
- moved P26 8.89 mm to (161.0, 72.1), turned to 270 degrees
- moved P27 8.89 mm to (161.0, 69.6), turned to 270 degrees
- moved P32 8.89 mm to (161.0, 64.8), turned to 270 degrees
- moved P33 8.89 mm to (161.0, 62.2), turned to 270 degrees
- moved P28 8.89 mm to (125.5, 72.3), turned to 270 degrees
- moved P29 8.89 mm to (125.5, 69.7), turned to 270 degrees
- moved P34 8.89 mm to (125.5, 64.8), turned to 270 degrees
- moved P35 8.89 mm to (125.5, 62.2), turned to 270 degrees
- moved P1 2.54 mm to (172.5, 72.1), turned to 270 degrees
- moved P13 2.54 mm to (172.5, 64.8), turned to 270 degrees
- moved P14 2.54 mm to (172.5, 62.2), turned to 270 degrees
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Connections:
- P39 pad 1: GND -> Net-(P39-Pad1)
- P40 pad 1: GND -> Net-(P40-Pad1)
Other:
- rule pad_to_mask_clearance: 0.254 -> 0.0762
