File: hardware/VR_ncv1124_test_module/ncv1124.sch (KiCad schematic (older format))
At the start: 34 parts, among them J1 Screw_Terminal_01x02, J2 Screw_Terminal_01x02, J3 Screw_Terminal_01x02, J4 Screw_Terminal_01x02, J5 Screw_Terminal_01x02, J6 Screw_Terminal_01x02, J7 Conn_01x02_Male, J8 Conn_01x03_Male, Q1 2N7002, Q2 2N7002

Commit message: ncv
Parts:
- added R14: 3K, Resistor_SMD:R_0805_2012Metric_Pad1.20x1.40mm_HandSolder, symbol Device:R
- D2: symbol ncv1124:NCV1124 -> ncv1124-rescue:NCV1124-ncv1124
- G1: symbol logo:LOGO -> ncv1124-rescue:LOGO-logo
- R1, R12, R13: value 160 -> 3K; LCSC C25269 -> C17661
Connections:
- wire segments 40 -> 41
Changed lines of the file:
@@
 P 2850 900
 F 0 "R1" V 2643 900 50  0000 C CNN
-F 1 "160" V 2734 900 50  0000 C CNN
+F 1 "3K" V 2734 900 50  0000 C CNN
 F 2 "Resistor_SMD:R_0805_2012Metric_Pad1.20x1.40mm_HandSolder" V 2780 900 50  0001 C CNN
 F 3 "~" H 2850 900 50  0001 C CNN
-F 4 "C25269" H 2850 900 50  0001 C CNN "LCSC"
+F 4 "C17661" H 2850 900 50  0001 C CNN "LCSC"
 	1    2850 900
 	0    1    1    0
@@
 	2400 900  2250 900
 $Comp
-L ncv1124:NCV1124 D2
+L ncv1124-rescue:NCV1124-ncv1124 D2
 U 1 1 5FD467DA
 P 4900 2600
@@
 P 8100 2550
 F 0 "R12" V 7893 2550 50  0000 C CNN
-F 1 "160" V 7984 2550 50  0000 C CNN
+F 1 "3K" V 7984 2550 50  0000 C CNN
 F 2 "Resistor_SMD:R_0805_2012Metric_Pad1.20x1.40mm_HandSolder" V 8030 2550 50  0001 C CNN
 F 3 "~" H 8100 2550 50  0001 C CNN
-F 4 "C25269" H 8100 2550 50  0001 C CNN "LCSC"
+F 4 "C17661" H 8100 2550 50  0001 C CNN "LCSC"
 	1    8100 2550
 	-1   0    0    1
@@
 P 8100 4000
 F 0 "R13" V 7893 4000 50  0000 C CNN
-F 1 "160" V 7984 4000 50  0000 C CNN
+F 1 "3K" V 7984 4000 50  0000 C CNN
 F 2 "Resistor_SMD:R_0805_2012Metric_Pad1.20x1.40mm_HandSolder" V 8030 4000 50  0001 C CNN
 F 3 "~" H 8100 4000 50  0001 C CNN
-F 4 "C25269" H 8100 4000 50  0001 C CNN "LCSC"
+F 4 "C17661" H 8100 4000 50  0001 C CNN "LCSC"
 	1    8100 4000
 	-1   0    0    1
@@
 	7400 4750 6650 4750
 Wire Wire Line
-	6650 4750 6650 3050
+	6650 4750 6650 4050
 Wire Wire Line
 	6650 3050 5950 3050
 $Comp
-L logo:LOGO G1
+L ncv1124-rescue:LOGO-logo G1
 U 1 1 5FDC6349
 P 1000 6550
@@
 	6850 3050 6650 3050
 Connection ~ 6650 3050
+$Comp
+L Device:R R14
+U 1 1 5FD7BDDC
+P 6500 4050
+F 0 "R14" V 6293 4050 50  0000 C CNN
+F 1 "3K" V 6384 4050 50  0000 C CNN
+F 2 "Resistor_SMD:R_0805_2012Metric_Pad1.20x1.40mm_HandSolder" V 6430 4050 50  0001 C CNN
+F 3 "~" H 6500 4050 50  0001 C CNN
+F 4 "C17661" H 6500 4050 50  0001 C CNN "LCSC"
+	1    6500 4050
+	0    -1   -1   0
+$EndComp
+Connection ~ 6650 4050
+Wire Wire Line
+	6650 4050 6650 3050
+$Comp
+L power:GND #PWR0124
+U 1 1 5FD7C306
+P 6350 4050
+F 0 "#PWR0124" H 6350 3800 50  0001 C CNN
+F 1 "GND" H 6355 3877 50  0000 C CNN
+F 2 "" H 6350 4050 50  0001 C CNN
+F 3 "" H 6350 4050 50  0001 C CNN
+	1    6350 4050
+	0    1    -1   0
+$EndComp
 $EndSCHEMATC
