File: hardware/Breakout_154pin_284617-1-Connector/284617-1.kicad_pcb (KiCad board)
At the start: 2 copper layers, 150 x 51.8 mm, 27 parts, among them P1 284617-1, P10 CONN_5, P11 CONN_9, P12 CONN_5, P13 CONN_9, P14 CONN_22, P15 CONN_22, P16 CONN_22, P17 CONN_22, P18 CONN_1, P19 CONN_1, P2 CONN_1, P20 CONN_1, P21 CONN_1, P22 CONN_1, P23 CONN_1, P24 CONN_1, P25 CONN_1, P3 CONN_1, P4 CONN_1, P5 CONN_1, P6 CONN_5, P7 CONN_9, P8 CONN_5, P9 CONN_9

Commit message: 154 progress
Parts:
- moved G? 3.27 mm to (82.0, 106.2) (x2)
Routing:
- net N-00000136: track 31.1 -> 133.7 mm
- net N-00000127: track 54.9 -> 74.8 mm
- net N-00000128: track 42.8 -> 55.0 mm
- net N-00000141: track 30.7 -> 36.6 mm
- net N-00000107: track 21.2 -> 25.8 mm
- net N-00000146: track 30.3 -> 34.6 mm
- net N-00000102: track 21.6 -> 25.9 mm
- net N-0000097: track 37.7 -> 41.0 mm
- net N-00000112: track 21.0 -> 22.8 mm
- net N-00000153: track 22.0 -> 23.6 mm
- net N-00000148: track 22.4 -> 21.9 mm
Other:
- rule trace_min: 0.254 -> 0.2
- board text added: "18"
- board text added: "2"
- board text added: "28"
- board text added: "29"
- board text added: "3"
- board text added: "4"
- board text added: "51"
- board text added: "6"
- board text added: "7"
- board text added: "72"
- board text added: "73"
- board text added: "94"
- board text added: "Connector 154pin rev0.3"
- board text added: "rusEFI.com"
- board text removed: "110"
- board text removed: "111"
- board text removed: "133"
- board text removed: "135"
- board text removed: "141"
- board text removed: "147"
- board text removed: "154"
- board text removed: "61"
- board text removed: "62"
- board text removed: "63"
- board text removed: "64"
- board text removed: "65"
- board text removed: "67"
- board text removed: "75"
- board text removed: "81"
- board text removed: "88"
- board text removed: "rusEFI.com R0.2"
